File: Placa de acionamento/Esquema 2 mosfets.brd (EAGLE design)
At the start: 66 x 57.2 mm, 22 parts, among them Q1 IRF540, Q2 IRF540, Q3 IRF540

Commit message: Placa de acionamento
Parts:
- removed Q3: IRF540, transistor-fet:TO220
- moved SP 17.8 mm to (30.5, 31.9), turned to 270 degrees
Connections:
- net BUZZER: now also SP.+; no longer Q3.1
- net GND: now also SP.-; no longer GND.P1, GND.P2, Q3.3
- net N$2: now also GND.P1, GND.P2; no longer Q3.2, SP.-
- net VCC: no longer SP.+
Routing:
- net N$2: track 32.8 -> 0.00 mm
- net VCC: track 83.2 -> 69.2 mm
- net BUZZER: track 20.7 -> 12.8 mm
Changed lines of the file:
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@@
 <drawing>
 <settings>
-<setting alwaysvectorfont="yes"/>
+<setting alwaysvectorfont="no"/>
 <setting verticaltext="up"/>
 </settings>
@@
 </layers>
 <board>
-<fusionsync huburn="a.YnVzaW5lc3M6ZGlzY2VudGU3MA" projecturn="a.YnVzaW5lc3M6ZGlzY2VudGU3MCMyMDIyMDIxNzQ5ODU5MDQ4MQ" f3durn="urn:adsk.wipprod:dm.lineage:RpODcveeSC6_xb2NUnBt0A" pcbguid="" lastpulledtime="" lastsyncedchangeguid="" latestrevisionid="d3c54600-be05-46a0-aa6c-7da2fb251511" lastsyncedrevisionid="d3c54600-be05-46a0-aa6c-7da2fb251511" lastboardhashguid="7a2e4fd7-505f-0dd0-e260-c932a55f449c" lastpushedtime="2023-08-13T06:55:43Z" linktopcb3d="true"/>
+<fusionsync huburn="a.YnVzaW5lc3M6ZGlzY2VudGU3MA" projecturn="a.YnVzaW5lc3M6ZGlzY2VudGU3MCMyMDIyMDIxNzQ5ODU5MDQ4MQ" f3durn="urn:adsk.wipprod:dm.lineage:RpODcveeSC6_xb2NUnBt0A" pcbguid="" lastpulledtime="" lastsyncedchangeguid="" latestrevisionid="d3c54600-be05-46a0-aa6c-7da2fb251511" lastsyncedrevisionid="d3c54600-be05-46a0-aa6c-7da2fb251511" lastboardhashguid="7a2e4fd7-505f-0dd0-e260-c932a55f449c" lastpushedtime="2023-08-13T06:55:43Z" linktopcb3d="false"/>
 <plain>
 <wire x1="0" y1="0" x2="66.02" y2="0" width="0" layer="20"/>
@@
 <attribute name="VALUE" x="51.943" y="29.21" size="1.778" layer="27" ratio="10"/>
 </element>
-<element name="Q3" library="transistor-fet" library_urn="urn:adsk.eagle:library:396" package="TO220" package3d_urn="urn:adsk.eagle:package:28520/1" value="IRF540" x="30.48" y="26.67" smashed="yes">
-<attribute name="NAME" x="26.67" y="31.877" size="1.778" layer="25" ratio="10"/>
-<attribute name="POPULARITY" value="5" x="72.39" y="17.78" size="1.778" layer="27" display="off"/>
-<attribute name="VALUE" x="26.543" y="29.21" size="1.778" layer="27" ratio="10"/>
-</element>
 <element name="R1" library="rcl" library_urn="urn:adsk.eagle:library:334" package="0207/10" package3d_urn="urn:adsk.eagle:package:23491/2" value="1k" x="10.541" y="51.308" smashed="yes">
 <attribute name="NAME" x="7.493" y="52.832" size="0.6096" layer="25" ratio="10"/>
@@
 <attribute name="VALUE" x="50.8" y="40.005" size="1.778" layer="27" ratio="10"/>
 </element>
-<element name="SP" library="buzzer" library_urn="urn:adsk.eagle:library:113" package="AL11P" package3d_urn="urn:adsk.eagle:package:5308/1" value="AL11P" x="29.21" y="49.657" smashed="yes" rot="R90">
-<attribute name="MF" value="" x="35.56" y="104.267" size="1.778" layer="27" rot="R90" display="off"/>
-<attribute name="MPN" value="" x="35.56" y="104.267" size="1.778" layer="27" rot="R90" display="off"/>
-<attribute name="NAME" x="22.86" y="46.482" size="0.6096" layer="25" ratio="10" rot="R90"/>
-<attribute name="OC_FARNELL" value="unknown" x="35.56" y="104.267" size="1.778" layer="27" rot="R90" display="off"/>
-<attribute name="OC_NEWARK" value="unknown" x="35.56" y="104.267" size="1.778" layer="27" rot="R90" display="off"/>
-<attribute name="POPULARITY" value="3" x="35.56" y="104.267" size="1.778" layer="27" rot="R90" display="off"/>
-<attribute name="VALUE" x="32.385" y="45.847" size="1.27" layer="27" ratio="10" rot="R90"/>
+<element name="SP" library="buzzer" library_urn="urn:adsk.eagle:library:113" package="AL11P" package3d_urn="urn:adsk.eagle:package:5308/1" value="AL11P" x="30.48" y="31.877" smashed="yes" rot="R270">
+<attribute name="MF" value="" x="24.13" y="-22.733" size="1.778" layer="27" rot="R270" display="off"/>
+<attribute name="MPN" value="" x="24.13" y="-22.733" size="1.778" layer="27" rot="R270" display="off"/>
+<attribute name="NAME" x="36.83" y="35.052" size="0.6096" layer="25" ratio="10" rot="R270"/>
+<attribute name="OC_FARNELL" value="unknown" x="24.13" y="-22.733" size="1.778" layer="27" rot="R270" display="off"/>
+<attribute name="OC_NEWARK" value="unknown" x="24.13" y="-22.733" size="1.778" layer="27" rot="R270" display="off"/>
+<attribute name="POPULARITY" value="3" x="24.13" y="-22.733" size="1.778" layer="27" rot="R270" display="off"/>
+<attribute name="VALUE" x="27.305" y="35.687" size="1.27" layer="27" ratio="10" rot="R270"/>
 </element>
 <element name="S1-S2" library="SparkFun-Connectors" package="1X02_2.54_SCREWTERM" value="" x="8.89" y="7.62" smashed="yes">
@@
 <signals>
 <signal name="BUZZER">
-<contactref element="Q3" pad="1"/>
 <wire x1="36.83" y1="7.62" x2="36.83" y2="8.89" width="1" layer="16"/>
 <wire x1="36.83" y1="8.89" x2="31.75" y2="13.97" width="1" layer="16"/>
-<wire x1="31.75" y1="13.97" x2="27.94" y2="17.78" width="1" layer="16"/>
-<wire x1="27.94" y1="17.78" x2="27.94" y2="20.32" width="1" layer="16"/>
 <contactref element="R4" pad="2"/>
 <contactref element="3.3-BUZ" pad="P1"/>
 <wire x1="29.21" y1="13.97" x2="31.75" y2="13.97" width="1" layer="16"/>
 <wire x1="27.94" y1="12.7" x2="29.21" y2="13.97" width="1.016" layer="16"/>
+<contactref element="SP" pad="+"/>
+<wire x1="31.75" y1="13.97" x2="30.48" y2="29.591" width="0" layer="19" extent="1-1"/>
 </signal>
 <signal name="GND">
@@
 <contactref element="BATERIA" pad="2"/>
 <contactref element="Q2" pad="3"/>
-<contactref element="Q3" pad="3"/>
 <contactref element="LSKIB1" pad="K"/>
 <contactref element="OP1" pad="2"/>
@@
 <contactref element="R3" pad="1"/>
 <contactref element="R2" pad="1"/>
-<contactref element="GND" pad="P2"/>
-<contactref element="GND" pad="P1"/>
+<contactref element="SP" pad="-"/>
+<wire x1="52.07" y1="41.91" x2="63.5" y2="49.53" width="0" layer="19" extent="1-1"/>
+<wire x1="38.1" y1="41.91" x2="52.07" y2="41.91" width="0" layer="19" extent="1-1"/>
+<wire x1="30.48" y1="34.163" x2="38.1" y2="41.91" width="0" layer="19" extent="1-1"/>
+<wire x1="17.78" y1="33.02" x2="30.48" y2="34.163" width="0" layer="19" extent="1-1"/>
+<wire x1="9.398" y1="35.941" x2="17.78" y2="33.02" width="0" layer="19" extent="1-1"/>
+<wire x1="7.62" y1="33.02" x2="9.398" y2="35.941" width="0" layer="19" extent="1-1"/>
+<wire x1="6.35" y1="43.18" x2="9.398" y2="35.941" width="0" layer="19" extent="1-1"/>
+<wire x1="7.62" y1="22.86" x2="7.62" y2="33.02" width="0" layer="19" extent="1-1"/>
+<wire x1="12.7" y1="16.51" x2="7.62" y2="22.86" width="0" layer="19" extent="1-1"/>
+<wire x1="17.78" y1="12.7" x2="12.7" y2="16.51" width="0" layer="19" extent="1-1"/>
+<wire x1="21.59" y1="7.62" x2="17.78" y2="12.7" width="0" layer="19" extent="1-1"/>
+<wire x1="21.59" y1="5.08" x2="21.59" y2="7.62" width="0" layer="19" extent="1-1"/>
+<wire x1="11.43" y1="53.34" x2="6.35" y2="43.18" width="0" layer="19" extent="1-1"/>
+<wire x1="20.32" y1="53.34" x2="11.43" y2="53.34" width="0" layer="19" extent="1-1"/>
+<wire x1="26.67" y1="48.26" x2="20.32" y2="53.34" width="0" layer="19" extent="1-1"/>
+<wire x1="33.02" y1="15.24" x2="21.59" y2="7.62" width="0" layer="19" extent="1-1"/>
+<wire x1="35.56" y1="13.97" x2="33.02" y2="15.24" width="0" layer="19" extent="1-1"/>
+<wire x1="36.83" y1="21.59" x2="33.02" y2="15.24" width="0" layer="19" extent="1-1"/>
+<wire x1="45.72" y1="20.32" x2="36.83" y2="21.59" width="0" layer="19" extent="1-1"/>
+<wire x1="49.53" y1="22.86" x2="45.72" y2="20.32" width="0" layer="19" extent="1-1"/>
+<wire x1="58.42" y1="20.32" x2="49.53" y2="22.86" width="0" layer="19" extent="1-1"/>
+<wire x1="58.42" y1="16.51" x2="58.42" y2="20.32" width="0" layer="19" extent="1-1"/>
+<wire x1="57.15" y1="13.97" x2="58.42" y2="16.51" width="0" layer="19" extent="1-1"/>
+<wire x1="62.23" y1="7.62" x2="57.15" y2="13.97" width="0" layer="19" extent="1-1"/>
+<wire x1="52.3494" y1="7.366" x2="57.15" y2="13.97" width="0" layer="19" extent="1-1"/>
 </signal>
 <signal name="SKIB1">
@@
 <contactref element="SKIB1" pad="1"/>
 <contactref element="SKIB2" pad="1"/>
-<contactref element="SP" pad="+"/>
 <wire x1="57.3786" y1="7.366" x2="57.3786" y2="10.3886" width="2.54" layer="1"/>
 <wire x1="62.23" y1="41.91" x2="59.69" y2="44.45" width="2.54" layer="1"/>
@@
 <wire x1="40.64" y1="45.72" x2="40.64" y2="49.53" width="2.54" layer="1"/>
 <wire x1="40.64" y1="49.53" x2="40.6654" y2="49.53" width="2.54" layer="1"/>
-<wire x1="40.64" y1="45.72" x2="36.83" y2="45.72" width="2.54" layer="1"/>
-<wire x1="30.607" y1="51.943" x2="29.21" y2="51.943" width="2.54" layer="1"/>
-<wire x1="36.83" y1="45.72" x2="30.607" y2="51.943" width="2.54" layer="1"/>
 </signal>
 <signal name="SKIB2">
@@
 <wire x1="48.26" y1="16.51" x2="50.8" y2="16.51" width="1.016" layer="16"/>
 <wire x1="50.8" y1="16.51" x2="52.07" y2="15.24" width="1.016" layer="16"/>
-</signal>
-<signal name="N$2">
-<contactref element="Q3" pad="2"/>
-<contactref element="SP" pad="-"/>
-<wire x1="29.21" y1="47.371" x2="36.83" y2="39.751" width="1.5" layer="16"/>
-<wire x1="36.83" y1="39.751" x2="36.83" y2="34.29" width="1.5" layer="16"/>
-<wire x1="36.83" y1="34.29" x2="30.48" y2="27.94" width="1.5" layer="16"/>
-<wire x1="30.48" y1="27.94" x2="30.48" y2="20.32" width="1.5" layer="16"/>
 </signal>
 <signal name="N$3">
@@
 <via x="10.16" y="41.91" extent="1-16" drill="0.35"/>
 </signal>
+<signal name="N$2">
+<contactref element="GND" pad="P2"/>
+<contactref element="GND" pad="P1"/>
+<wire x1="16.51" y1="7.62" x2="19.05" y2="7.62" width="0" layer="19" extent="1-1"/>
+</signal>
 </signals>
