File: Placa de acionamento/Esquema Acionamento 01/Esquema 01 guilherme.brd (EAGLE design)
At the start: 66 x 57.2 mm, 22 parts, among them Q1 IRF540, Q2 IRF540, Q3 IRF540

Commit message: Placa de acionamento
Parts:
- BATERIA, SKIB1, SKIB2: device con-ptr500:AK500/2-H -> SparkFun-Connectors:1X02_2.54_SCREWTERM
- moved SKIB2 15.2 mm to (40.6, 49.5)
- moved 3.3-BUZ 7.62 mm to (26.7, 7.62)
- moved SKIB1 6.35 mm to (49.5, 49.5)
- moved BATERIA 4.07 mm to (50.8, 7.62), turned to 0 degrees
- moved R4 1.80 mm to (24.1, 14.0)
- moved LSKIB1 1.27 mm to (10.7, 34.7)
- moved Q1 1.27 mm to (44.5, 26.7)
- moved SK1-SK2 1.27 mm to (41.9, 7.62)
- moved GND 1.27 mm to (17.8, 7.62)
- moved Q3 1.27 mm to (31.8, 26.7)
- moved Q2 1.27 mm to (57.1, 26.7)
Connections:
- net GND: now also BATERIA.P1; no longer BATERIA.2
- net SKIB1_CONECTOR: now also SKIB1.P1; no longer SKIB1.2
- net SKIB2_CONECTOR: now also SKIB2.P1; no longer SKIB2.2
- net VCC: now also BATERIA.P2, SKIB1.P2, SKIB2.P2; no longer BATERIA.1, SKIB1.1, SKIB2.1
Routing:
- net SKIB2_CONECTOR: track 95.0 -> 111.3 mm
- net BUZZER: track 20.7 -> 12.7 mm
- net 3.3V: track 61.9 -> 54.3 mm
- net VCC: track 83.2 -> 87.5 mm
- net SKIB2: track 20.2 -> 22.0 mm
- net SKIB1: track 17.6 -> 16.5 mm
- net SKIB1_CONECTOR: track 94.2 -> 93.6 mm
- net N$3: track 6.74 -> 7.26 mm
- net N$2: track 32.8 -> 32.3 mm
