File: Placa de acionamento/Esquema Acionamento 01/Esquema 01 guilherme.sch (EAGLE design)
At the start: 22 parts, among them Q1 IRF540, Q2 IRF540, Q3 IRF540

Commit message: Placa de acionamento
Parts:
- BATERIA, SKIB1, SKIB2: device con-ptr500:AK500/2-H -> SparkFun-Connectors:CONN_022.54MM_SCREWTERM
Connections:
- net GND: now also BATERIA.1; no longer BATERIA-2.KL
- net SKIB1_CONECTOR: now also SKIB1.1; no longer SKIB1-2.KL
- net SKIB2_CONECTOR: now also SKIB2.1; no longer SKIB2-2.KL
- net VCC: now also BATERIA.2, SKIB1.2, SKIB2.2; no longer BATERIA-1.KL, SKIB1-1.KL, SKIB2-1.KL
Changed lines of the file:
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@@
 <drawing>
 <settings>
-<setting alwaysvectorfont="yes"/>
+<setting alwaysvectorfont="no"/>
 <setting verticaltext="up"/>
 </settings>
@@
 <part name="Q1" library="transistor-fet" library_urn="urn:adsk.eagle:library:396" deviceset="IRF540" device="" package3d_urn="urn:adsk.eagle:package:28520/1"/>
 <part name="GND6" library="supply1" library_urn="urn:adsk.eagle:library:371" deviceset="GND" device=""/>
-<part name="BATERIA" library="con-ptr500" library_urn="urn:adsk.eagle:library:181" deviceset="AK500/2-H" device="" package3d_urn="urn:adsk.eagle:package:9901/1"/>
 <part name="GND10" library="supply1" library_urn="urn:adsk.eagle:library:371" deviceset="GND" device=""/>
-<part name="SKIB1" library="con-ptr500" library_urn="urn:adsk.eagle:library:181" deviceset="AK500/2-H" device="" package3d_urn="urn:adsk.eagle:package:9901/1"/>
 <part name="P+3" library="supply1" library_urn="urn:adsk.eagle:library:371" deviceset="VCC" device=""/>
 <part name="P+1" library="supply1" library_urn="urn:adsk.eagle:library:371" deviceset="VCC" device=""/>
 <part name="Q2" library="transistor-fet" library_urn="urn:adsk.eagle:library:396" deviceset="IRF540" device="" package3d_urn="urn:adsk.eagle:package:28520/1"/>
 <part name="GND8" library="supply1" library_urn="urn:adsk.eagle:library:371" deviceset="GND" device=""/>
-<part name="SKIB2" library="con-ptr500" library_urn="urn:adsk.eagle:library:181" deviceset="AK500/2-H" device="" package3d_urn="urn:adsk.eagle:package:9901/1"/>
 <part name="P+2" library="supply1" library_urn="urn:adsk.eagle:library:371" deviceset="VCC" device=""/>
 <part name="Q3" library="transistor-fet" library_urn="urn:adsk.eagle:library:396" deviceset="IRF540" device="" package3d_urn="urn:adsk.eagle:package:28520/1"/>
@@
 <part name="GND" library="SparkFun-Connectors" deviceset="CONN_02" device="2.54MM_SCREWTERM"/>
 <part name="GND12" library="supply1" library_urn="urn:adsk.eagle:library:371" deviceset="GND" device=""/>
+<part name="BATERIA" library="SparkFun-Connectors" deviceset="CONN_02" device="2.54MM_SCREWTERM"/>
+<part name="SKIB1" library="SparkFun-Connectors" deviceset="CONN_02" device="2.54MM_SCREWTERM"/>
+<part name="SKIB2" library="SparkFun-Connectors" deviceset="CONN_02" device="2.54MM_SCREWTERM"/>
 </parts>
 <sheets>
@@
 <attribute name="VALUE" x="66.04" y="55.88" size="1.778" layer="96"/>
 </instance>
-<instance part="BATERIA" gate="-1" x="-7.62" y="60.96" smashed="yes">
-<attribute name="NAME" x="-8.89" y="61.849" size="1.778" layer="95" rot="R180"/>
-</instance>
-<instance part="BATERIA" gate="-2" x="-7.62" y="55.88" smashed="yes">
-<attribute name="NAME" x="-8.89" y="56.769" size="1.778" layer="95" rot="R180"/>
-<attribute name="VALUE" x="-11.43" y="52.197" size="1.778" layer="96"/>
-</instance>
 <instance part="GND10" gate="1" x="2.54" y="50.8" smashed="yes">
 <attribute name="VALUE" x="0" y="48.26" size="1.778" layer="96"/>
-</instance>
-<instance part="SKIB1" gate="-1" x="48.26" y="83.82" smashed="yes">
-<attribute name="NAME" x="46.99" y="84.709" size="1.778" layer="95" rot="R180"/>
-</instance>
-<instance part="SKIB1" gate="-2" x="48.26" y="78.74" smashed="yes">
-<attribute name="NAME" x="46.99" y="79.629" size="1.778" layer="95" rot="R180"/>
-<attribute name="VALUE" x="44.45" y="75.057" size="1.778" layer="96"/>
 </instance>
 <instance part="P+3" gate="VCC" x="68.58" y="93.98" smashed="yes">
@@
 <attribute name="VALUE" x="66.04" y="0" size="1.778" layer="96"/>
 </instance>
-<instance part="SKIB2" gate="-1" x="48.26" y="27.94" smashed="yes">
-<attribute name="NAME" x="46.99" y="28.829" size="1.778" layer="95" rot="R180"/>
-</instance>
-<instance part="SKIB2" gate="-2" x="48.26" y="22.86" smashed="yes">
-<attribute name="NAME" x="46.99" y="23.749" size="1.778" layer="95" rot="R180"/>
-<attribute name="VALUE" x="44.45" y="19.177" size="1.778" layer="96"/>
-</instance>
 <instance part="P+2" gate="VCC" x="68.58" y="38.1" smashed="yes">
 <attribute name="VALUE" x="66.04" y="35.56" size="1.778" layer="96" rot="R90"/>
@@
 <instance part="GND12" gate="1" x="149.86" y="81.28" smashed="yes">
 <attribute name="VALUE" x="147.32" y="78.74" size="1.778" layer="96"/>
+</instance>
+<instance part="BATERIA" gate="G$1" x="-10.16" y="55.88" smashed="yes">
+<attribute name="VALUE" x="-12.7" y="51.054" size="1.778" layer="96" font="vector"/>
+<attribute name="NAME" x="-12.7" y="61.468" size="1.778" layer="95" font="vector"/>
+</instance>
+<instance part="SKIB1" gate="G$1" x="45.72" y="81.28" smashed="yes">
+<attribute name="VALUE" x="43.18" y="76.454" size="1.778" layer="96" font="vector"/>
+<attribute name="NAME" x="43.18" y="86.868" size="1.778" layer="95" font="vector"/>
+</instance>
+<instance part="SKIB2" gate="G$1" x="45.72" y="25.4" smashed="yes">
+<attribute name="VALUE" x="43.18" y="20.574" size="1.778" layer="96" font="vector"/>
+<attribute name="NAME" x="43.18" y="30.988" size="1.778" layer="95" font="vector"/>
 </instance>
 </instances>
@@
 </segment>
 <segment>
-<pinref part="BATERIA" gate="-2" pin="KL"/>
 <pinref part="GND10" gate="1" pin="GND"/>
 <wire x1="-2.54" y1="55.88" x2="2.54" y2="55.88" width="0.1524" layer="91"/>
 <wire x1="2.54" y1="55.88" x2="2.54" y2="53.34" width="0.1524" layer="91"/>
+<pinref part="BATERIA" gate="G$1" pin="1"/>
 </segment>
 <segment>
@@
 <net name="VCC" class="0">
 <segment>
-<pinref part="BATERIA" gate="-1" pin="KL"/>
-<wire x1="-2.54" y1="60.96" x2="2.54" y2="60.96" width="0.1524" layer="91"/>
+<wire x1="-2.54" y1="58.42" x2="2.54" y2="58.42" width="0.1524" layer="91"/>
 <pinref part="P+1" gate="VCC" pin="VCC"/>
-<wire x1="2.54" y1="60.96" x2="2.54" y2="66.04" width="0.1524" layer="91"/>
+<wire x1="2.54" y1="58.42" x2="2.54" y2="66.04" width="0.1524" layer="91"/>
+<pinref part="BATERIA" gate="G$1" pin="2"/>
 </segment>
 <segment>
 <pinref part="P+3" gate="VCC" pin="VCC"/>
 <wire x1="68.58" y1="91.44" x2="68.58" y2="86.36" width="0.1524" layer="91"/>
-<pinref part="SKIB1" gate="-1" pin="KL"/>
 <wire x1="53.34" y1="83.82" x2="58.42" y2="83.82" width="0.1524" layer="91"/>
 <wire x1="58.42" y1="83.82" x2="58.42" y2="86.36" width="0.1524" layer="91"/>
 <wire x1="58.42" y1="86.36" x2="68.58" y2="86.36" width="0.1524" layer="91"/>
 <label x="58.42" y="86.36" size="1.778" layer="95"/>
+<pinref part="SKIB1" gate="G$1" pin="2"/>
 </segment>
 <segment>
 <pinref part="P+2" gate="VCC" pin="VCC"/>
 <wire x1="68.58" y1="35.56" x2="68.58" y2="30.48" width="0.1524" layer="91"/>
-<pinref part="SKIB2" gate="-1" pin="KL"/>
 <wire x1="53.34" y1="27.94" x2="58.42" y2="27.94" width="0.1524" layer="91"/>
 <wire x1="58.42" y1="27.94" x2="58.42" y2="30.48" width="0.1524" layer="91"/>
 <wire x1="58.42" y1="30.48" x2="68.58" y2="30.48" width="0.1524" layer="91"/>
 <label x="58.42" y="30.48" size="1.778" layer="95"/>
+<pinref part="SKIB2" gate="G$1" pin="2"/>
 </segment>
 <segment>
@@
 <wire x1="68.58" y1="71.12" x2="68.58" y2="76.2" width="0.1524" layer="91"/>
 <wire x1="58.42" y1="76.2" x2="68.58" y2="76.2" width="0.1524" layer="91"/>
-<pinref part="SKIB1" gate="-2" pin="KL"/>
-<wire x1="53.34" y1="78.74" x2="58.42" y2="78.74" width="0.1524" layer="91"/>
-<wire x1="58.42" y1="78.74" x2="58.42" y2="76.2" width="0.1524" layer="91"/>
+<wire x1="53.34" y1="81.28" x2="58.42" y2="81.28" width="0.1524" layer="91"/>
+<wire x1="58.42" y1="81.28" x2="58.42" y2="76.2" width="0.1524" layer="91"/>
 <label x="58.42" y="76.2" size="1.778" layer="95"/>
 <pinref part="Q1" gate="G$1" pin="D"/>
+<pinref part="SKIB1" gate="G$1" pin="1"/>
 </segment>
 </net>
@@
 <wire x1="68.58" y1="15.24" x2="68.58" y2="20.32" width="0.1524" layer="91"/>
 <wire x1="58.42" y1="20.32" x2="68.58" y2="20.32" width="0.1524" layer="91"/>
-<pinref part="SKIB2" gate="-2" pin="KL"/>
-<wire x1="53.34" y1="22.86" x2="58.42" y2="22.86" width="0.1524" layer="91"/>
-<wire x1="58.42" y1="22.86" x2="58.42" y2="20.32" width="0.1524" layer="91"/>
+<wire x1="53.34" y1="25.4" x2="58.42" y2="25.4" width="0.1524" layer="91"/>
+<wire x1="58.42" y1="25.4" x2="58.42" y2="20.32" width="0.1524" layer="91"/>
 <label x="58.42" y="20.32" size="1.778" layer="95"/>
 <pinref part="Q2" gate="G$1" pin="D"/>
-</segment>
-</net>
+<pinref part="SKIB2" gate="G$1" pin="1"/>
+</segment>
+</net>
