File: Placa de acionamento/Esquema Acionamento 01/Esquema 02 guilherme.sch (EAGLE design)
At the start: 22 parts, among them Q1 IRF540, Q2 IRF540, Q3 IRF540

Commit message: Placa de acionamento
Parts:
- removed Q3: IRF540, transistor-fet:IRF540
- BATERIA, SKIB1, SKIB2: device con-ptr500:AK500/2-H -> SparkFun-Connectors:CONN_022.54MM_SCREWTERM
Connections:
- removed net N$2: Q3.D, SP.1
- net BUZZER: now also SP.2; no longer Q3.G
- net GND: now also BATERIA.1, SP.1; no longer BATERIA-2.KL, Q3.S
- net SKIB1_CONECTOR: now also SKIB1.1; no longer SKIB1-2.KL
- net SKIB2_CONECTOR: now also SKIB2.1; no longer SKIB2-2.KL
- net VCC: now also BATERIA.2, SKIB1.2, SKIB2.2; no longer BATERIA-1.KL, SKIB1-1.KL, SKIB2-1.KL, SP.2
