File: Placa de acionamento/Esquema Acionamento 01/Esquema 03 guilherme.brd (EAGLE design)
At the start: 80 x 47 mm, 21 parts, among them Q1 IRF540, Q2 IRF540

Commit message: Finalizados os ajustes na placa de acionamento do Joliot.
Parts:
- moved R7 4.24 mm to (37.4, 24.1)
- moved R2 1.00 mm to (43.5, 24.1)
Routing:
- net GND: track 0.00 -> 196.3 mm, vias 6 -> 10
- net 3.3V: track 21.3 -> 41.6 mm, vias 0 -> 2
- net SKIB2_CONECTOR: track 52.9 -> 64.4 mm, vias 0 -> 1
- net SKIB2: track 97.3 -> 99.9 mm
- net N$1: track 2.77 -> 4.96 mm, vias 1 -> 0
- net SINAL_SKIB1: track 18.8 -> 20.5 mm
- net VCC: track 24.1 -> 25.3 mm
- net SKIB1_CONECTOR: track 64.9 -> 64.1 mm
