File: Placa de processamento - antiga/Esquema.brd (EAGLE design)
At the start: 145.1 x 90.2 mm, 12 parts

Commit message: Roteamento da placa
Parts:
- removed IC1: (no value), v-reg:78LXX
- moved U$2 16.6 mm to (123.2, 57.1)
- moved U$10 9.25 mm to (7.62, 16.5)
- moved U$11 2.84 mm to (109.2, 17.8)
- moved U$4 2.54 mm to (26.7, 17.8)
- moved U$6 2.54 mm to (19.1, 17.8)
- moved U$3 1.27 mm to (73.7, 21.6), turned to 180 degrees
- turned U$5 to 90 degrees
- turned U$7 to 90 degrees
Connections:
- removed net GND: U$11.29, U$7.2
- removed net N$12: IC1.OUT, U$2.VCC
- removed net N$15: U$11.9, U$8.CLK
- removed net N$16: U$11.10, U$8.MISO
- removed net N$19: U$11.28, U$6.1
- removed net N$20: U$11.27, U$6.2
- removed net N$21: U$11.26, U$4.1
- removed net N$22: U$11.19, U$5.1
- removed net N$23: U$11.20, U$5.2
- removed net V_BATTERY: U$10.PL3, U$10.PR3, U$7.1
- net N$1: now also U$11.21; no longer U$11.11
- net N$10: now also U$11.19, U$8.MISO; no longer U$11.22, U$2.M1
- net N$11: now also U$10.PR2, U$11.30; no longer U$11.21, U$2.M0
- net N$13: now also U$11.17, U$2.RXD; no longer U$11.8, U$8.CS
- net N$14: now also U$11.16, U$2.TXD; no longer U$11.15, U$8.MOSI
- net N$2: now also U$11.22; no longer U$11.14
- net N$3: no longer U$4.2
- net N$4: no longer IC1.GND
- net N$5: now also U$11.15, U$3.TX; no longer U$11.5, U$3.RX
- net N$6: now also U$11.4, U$3.RX; no longer U$11.3, U$3.TX
- net N$7: now also U$11.5, U$8.CS; no longer IC1.IN, U$10.PL2, U$10.PR2, U$11.30
- net N$8: now also U$11.23, U$8.MOSI; no longer U$11.7, U$2.TXD
- net N$9: now also U$11.18, U$8.CLK; no longer U$11.6, U$2.RXD
Routing:
- net N$7: track 220.8 -> 0.00 mm, vias 2 -> 0
- net N$20: track 130.1 -> 0.00 mm, vias 1 -> 0
- net N$3: track 109.8 -> 0.00 mm
- net N$11: track 99.8 -> 0.00 mm
- net N$2: track 94.7 -> 0.00 mm
- net N$13: track 89.9 -> 0.00 mm
- net N$23: track 89.4 -> 0.00 mm
- net N$15: track 88.5 -> 0.00 mm, vias 2 -> 0
- net N$1: track 87.1 -> 0.00 mm
- net N$16: track 85.7 -> 0.00 mm, vias 2 -> 0
- net N$12: track 82.7 -> 0.00 mm
- net N$10: track 78.2 -> 0.00 mm
- net N$14: track 74.3 -> 0.00 mm, vias 2 -> 0
- net N$6: track 68.0 -> 0.00 mm, vias 2 -> 0
- net N$5: track 61.7 -> 0.00 mm
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Other:
- board size 145.1 x 90.2 mm -> 145.1 x 71.2 mm
