File: Placa de processamento/Esquema.sch (EAGLE design)
At the start: 12 parts

Commit message: Componentes de biblioteca atualizados
Changed lines of the file:
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@@
 </classes>
 <parts>
-<part name="U$1" library="CRD" library_urn="urn:adsk.eagle:library:39051337" deviceset="BMP390" device="V1" package3d_urn="urn:adsk.eagle:package:40965124/4"/>
-<part name="U$2" library="CRD" library_urn="urn:adsk.eagle:library:39051337" deviceset="E22-400T30D" device="" package3d_urn="urn:adsk.eagle:package:40965099/3"/>
-<part name="U$3" library="CRD" library_urn="urn:adsk.eagle:library:39051337" deviceset="GPS_MODULE" device="" package3d_urn="urn:adsk.eagle:package:39608400/4"/>
+<part name="U$1" library="CRD" library_urn="urn:adsk.eagle:library:39051337" deviceset="BMP390" device="V1" package3d_urn="urn:adsk.eagle:package:40965124/5"/>
+<part name="U$2" library="CRD" library_urn="urn:adsk.eagle:library:39051337" deviceset="E22-400T30D" device="" package3d_urn="urn:adsk.eagle:package:40965099/4"/>
+<part name="U$3" library="CRD" library_urn="urn:adsk.eagle:library:39051337" deviceset="GPS_MODULE" device="" package3d_urn="urn:adsk.eagle:package:39608400/5"/>
 <part name="U$4" library="CRD" library_urn="urn:adsk.eagle:library:39051337" deviceset="JST2.54X2P" device="" package3d_urn="urn:adsk.eagle:package:39191967/2"/>
 <part name="U$5" library="CRD" library_urn="urn:adsk.eagle:library:39051337" deviceset="JST2.54X2P" device="" package3d_urn="urn:adsk.eagle:package:39191967/2"/>
 <part name="U$6" library="CRD" library_urn="urn:adsk.eagle:library:39051337" deviceset="JST2.54X2P" device="" package3d_urn="urn:adsk.eagle:package:39191967/2"/>
 <part name="U$7" library="CRD" library_urn="urn:adsk.eagle:library:39051337" deviceset="JST2.54X2P" device="" package3d_urn="urn:adsk.eagle:package:39191967/2"/>
-<part name="U$10" library="CRD" library_urn="urn:adsk.eagle:library:39051337" deviceset="PRESSION_BUTTON" device="" package3d_urn="urn:adsk.eagle:package:43483815/1"/>
+<part name="U$10" library="CRD" library_urn="urn:adsk.eagle:library:39051337" deviceset="PRESSION_BUTTON" device="" package3d_urn="urn:adsk.eagle:package:43483815/3"/>
 <part name="U$8" library="CRD" library_urn="urn:adsk.eagle:library:39051337" deviceset="MICROSD_SMALL_READER" device="" package3d_urn="urn:adsk.eagle:package:44017969/2"/>
-<part name="U$9" library="CRD" library_urn="urn:adsk.eagle:library:39051337" deviceset="MPU6050" device="V1" package3d_urn="urn:adsk.eagle:package:39029071/7"/>
+<part name="U$9" library="CRD" library_urn="urn:adsk.eagle:library:39051337" deviceset="MPU6050" device="V1" package3d_urn="urn:adsk.eagle:package:39029071/8"/>
 <part name="U$11" library="ESP32-DEVKITV1" library_urn="urn:adsk.eagle:library:44018017" deviceset="ESP32DEVKITV1" device="" package3d_urn="urn:adsk.eagle:package:44018021/1"/>
 <part name="IC1" library="v-reg" library_urn="urn:adsk.eagle:library:409" deviceset="78LXX" device="" package3d_urn="urn:adsk.eagle:package:30346/1"/>
@@
 <wire x1="48.26" y1="40.64" x2="48.26" y2="35.56" width="0.1524" layer="91"/>
 <junction x="48.26" y="35.56"/>
+<pinref part="U$10" gate="G$1" pin="PR2"/>
+<wire x1="-2.54" y1="73.66" x2="-2.54" y2="40.64" width="0.1524" layer="91"/>
+<wire x1="-29.21" y1="43.18" x2="-29.21" y2="40.64" width="0.1524" layer="91"/>
+<wire x1="-29.21" y1="40.64" x2="-2.54" y2="40.64" width="0.1524" layer="91"/>
+<junction x="-2.54" y="40.64"/>
 <pinref part="U$10" gate="G$1" pin="PL2"/>
-<wire x1="-28.194" y1="78.74" x2="-2.54" y2="78.74" width="0.1524" layer="91"/>
-<wire x1="-2.54" y1="78.74" x2="-2.54" y2="40.64" width="0.1524" layer="91"/>
-<wire x1="-28.194" y1="64.77" x2="-28.194" y2="78.74" width="0.1524" layer="91"/>
-<pinref part="U$10" gate="G$1" pin="PR2"/>
-<wire x1="-30.734" y1="46.99" x2="-30.734" y2="40.64" width="0.1524" layer="91"/>
-<wire x1="-30.734" y1="40.64" x2="-2.54" y2="40.64" width="0.1524" layer="91"/>
-<junction x="-2.54" y="40.64"/>
+<wire x1="-29.21" y1="68.58" x2="-29.21" y2="73.66" width="0.1524" layer="91"/>
+<wire x1="-29.21" y1="73.66" x2="-2.54" y2="73.66" width="0.1524" layer="91"/>
 </segment>
 </net>
@@
 <pinref part="U$7" gate="G$1" pin="1"/>
 <wire x1="10.16" y1="71.12" x2="27.94" y2="71.12" width="0.1524" layer="91"/>
-<wire x1="-33.274" y1="73.66" x2="-43.18" y2="73.66" width="0.1524" layer="91"/>
+<wire x1="-34.29" y1="73.66" x2="-43.18" y2="73.66" width="0.1524" layer="91"/>
 <wire x1="-43.18" y1="73.66" x2="-43.18" y2="40.64" width="0.1524" layer="91"/>
 <label x="10.16" y="58.42" size="1.27" layer="95" rot="R90"/>
 <pinref part="U$10" gate="G$1" pin="PL3"/>
 <wire x1="-43.18" y1="40.64" x2="-43.18" y2="38.1" width="0.1524" layer="91"/>
-<wire x1="-33.274" y1="64.77" x2="-33.274" y2="73.66" width="0.1524" layer="91"/>
+<wire x1="-34.29" y1="40.64" x2="-43.18" y2="40.64" width="0.1524" layer="91"/>
+<junction x="-43.18" y="40.64"/>
+<wire x1="-34.29" y1="68.58" x2="-34.29" y2="73.66" width="0.1524" layer="91"/>
 <pinref part="U$10" gate="G$1" pin="PR3"/>
-<wire x1="-35.814" y1="46.99" x2="-35.56" y2="46.99" width="0.1524" layer="91"/>
-<wire x1="-35.56" y1="46.99" x2="-35.56" y2="40.64" width="0.1524" layer="91"/>
-<wire x1="-35.56" y1="40.64" x2="-43.18" y2="40.64" width="0.1524" layer="91"/>
-<junction x="-43.18" y="40.64"/>
-</segment>
-</net>
+<wire x1="-34.29" y1="43.18" x2="-34.29" y2="40.64" width="0.1524" layer="91"/>
+</segment>
+</net>

Commit message: Ajustes na PCB finalizados!
Connections:
- removed net N$4: IC1.GND, U$1.GND, U$11.GND, U$2.GND, U$3.GND, U$8.GND, U$9.GND
- net GND: now also IC1.GND, U$1.GND, U$11.GND, U$2.GND, U$3.GND, U$8.GND, U$9.GND
Changed lines of the file:
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@@
-</segment>
-</net>
-<net name="N$4" class="0">
-<segment>
-<pinref part="U$11" gate="G$1" pin="GND"/>
-<wire x1="50.8" y1="0" x2="50.8" y2="-2.54" width="0.1524" layer="91"/>
-<wire x1="50.8" y1="-2.54" x2="50.8" y2="-5.08" width="0.1524" layer="91"/>
-<wire x1="50.8" y1="-5.08" x2="50.8" y2="-15.24" width="0.1524" layer="91"/>
-<wire x1="50.8" y1="-15.24" x2="137.16" y2="-15.24" width="0.1524" layer="91"/>
-<pinref part="U$9" gate="G$1" pin="GND"/>
-<wire x1="137.16" y1="-15.24" x2="177.8" y2="-15.24" width="0.1524" layer="91"/>
-<wire x1="177.8" y1="-15.24" x2="177.8" y2="43.18" width="0.1524" layer="91"/>
-<pinref part="U$1" gate="G$1" pin="GND"/>
-<wire x1="137.16" y1="45.72" x2="137.16" y2="-15.24" width="0.1524" layer="91"/>
-<junction x="137.16" y="-15.24"/>
-<pinref part="U$3" gate="G$1" pin="GND"/>
-<wire x1="30.48" y1="-27.94" x2="50.8" y2="-27.94" width="0.1524" layer="91"/>
-<wire x1="50.8" y1="-27.94" x2="50.8" y2="-15.24" width="0.1524" layer="91"/>
-<junction x="50.8" y="-15.24"/>
-<pinref part="IC1" gate="1" pin="GND"/>
-<wire x1="7.62" y1="20.32" x2="7.62" y2="-5.08" width="0.1524" layer="91"/>
-<wire x1="7.62" y1="-5.08" x2="50.8" y2="-5.08" width="0.1524" layer="91"/>
-<junction x="50.8" y="-5.08"/>
-<pinref part="U$8" gate="G$1" pin="GND"/>
-<wire x1="147.32" y1="-53.34" x2="50.8" y2="-53.34" width="0.1524" layer="91"/>
-<wire x1="50.8" y1="-53.34" x2="50.8" y2="-27.94" width="0.1524" layer="91"/>
-<junction x="50.8" y="-27.94"/>
-<pinref part="U$2" gate="G$1" pin="GND"/>
-<wire x1="0" y1="0" x2="20.32" y2="0" width="0.1524" layer="91"/>
-<wire x1="20.32" y1="0" x2="20.32" y2="-2.54" width="0.1524" layer="91"/>
-<wire x1="20.32" y1="-2.54" x2="50.8" y2="-2.54" width="0.1524" layer="91"/>
-<junction x="50.8" y="-2.54"/>
 </segment>
 </net>
@@
 <label x="33.02" y="60.96" size="1.27" layer="95" rot="R90"/>
 </segment>
-</net>
+<segment>
+<pinref part="U$11" gate="G$1" pin="GND"/>
+<wire x1="50.8" y1="0" x2="50.8" y2="-2.54" width="0.1524" layer="91"/>
+<wire x1="50.8" y1="-2.54" x2="50.8" y2="-5.08" width="0.1524" layer="91"/>
+<wire x1="50.8" y1="-5.08" x2="50.8" y2="-15.24" width="0.1524" layer="91"/>
+<wire x1="50.8" y1="-15.24" x2="137.16" y2="-15.24" width="0.1524" layer="91"/>
+<pinref part="U$9" gate="G$1" pin="GND"/>
+<wire x1="137.16" y1="-15.24" x2="177.8" y2="-15.24" width="0.1524" layer="91"/>
+<wire x1="177.8" y1="-15.24" x2="177.8" y2="43.18" width="0.1524" layer="91"/>
+<pinref part="U$1" gate="G$1" pin="GND"/>
+<wire x1="137.16" y1="45.72" x2="137.16" y2="-15.24" width="0.1524" layer="91"/>
+<junction x="137.16" y="-15.24"/>
+<junction x="50.8" y="-15.24"/>
+<pinref part="IC1" gate="1" pin="GND"/>
+<wire x1="7.62" y1="20.32" x2="7.62" y2="-5.08" width="0.1524" layer="91"/>
+<wire x1="7.62" y1="-5.08" x2="50.8" y2="-5.08" width="0.1524" layer="91"/>
+<junction x="50.8" y="-5.08"/>
+<pinref part="U$8" gate="G$1" pin="GND"/>
+<wire x1="147.32" y1="-53.34" x2="50.8" y2="-53.34" width="0.1524" layer="91"/>
+<wire x1="50.8" y1="-53.34" x2="50.8" y2="-15.24" width="0.1524" layer="91"/>
+<pinref part="U$2" gate="G$1" pin="GND"/>
+<wire x1="0" y1="0" x2="20.32" y2="0" width="0.1524" layer="91"/>
+<wire x1="20.32" y1="0" x2="20.32" y2="-2.54" width="0.1524" layer="91"/>
+<junction x="50.8" y="-2.54"/>
+<wire x1="20.32" y1="-2.54" x2="50.8" y2="-2.54" width="0.1524" layer="91"/>
+<pinref part="U$3" gate="G$1" pin="GND"/>
+<wire x1="30.48" y1="-27.94" x2="30.48" y2="-15.24" width="0.1524" layer="91"/>
+<wire x1="30.48" y1="-15.24" x2="50.8" y2="-15.24" width="0.1524" layer="91"/>
+</segment>
+</net>
