File: Placa de baterias/Versões/Versão 2/Esquema.brd (EAGLE design)
At the start: 35.6 x 24.4 mm, 6 parts

Commit message: atualização placa de baterias
Parts:
- removed V: 22-23-2041, con-molex:22-23-2041
- added X1: 5566-4, con-molex:5566-4
- moved U$4 1.27 mm to (22.9, 12.7)
- moved U$5 1.27 mm to (12.7, 12.7)
Connections:
- net V1+: now also X1.3; no longer V.3
- net V1-: now also X1.1; no longer V.4
- net V2+: now also X1.2; no longer V.2
- net V2-: now also X1.4; no longer V.1
Routing:
- net V1+: track 34.0 -> 23.4 mm
- net V2-: track 23.5 -> 31.8 mm
- net V2+: track 29.0 -> 31.5 mm
- net V1-: track 15.3 -> 16.8 mm
Other:
- board size 35.6 x 24.4 mm -> 35.6 x 40.6 mm
