File: Placa de baterias/Versões/Versão 1/Esquema.brd (EAGLE design)
At the start: 35.6 x 24.4 mm, 6 parts

Commit message: placa de baterias
Parts:
- moved U$5 0.65 mm to (12.8, 12.1)
- moved U$4 0.63 mm to (22.9, 12.1)
Changed lines of the file:
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@@
 <element name="U$2" library="CRD" library_urn="urn:adsk.eagle:library:39051337" package="JST2.54X2P_FOOTPRINT" package3d_urn="urn:adsk.eagle:package:39191967/2" value="JST2.54X2P" x="17.78" y="5.08" smashed="yes" rot="R180"/>
 <element name="U$3" library="CRD" library_urn="urn:adsk.eagle:library:39051337" package="JST2.54X2P_FOOTPRINT" package3d_urn="urn:adsk.eagle:package:39191967/2" value="JST2.54X2P" x="8.89" y="5.08" smashed="yes" rot="R180"/>
-<element name="U$4" library="CRD" library_urn="urn:adsk.eagle:library:39051337" package="JST2.54X2P_FOOTPRINT" package3d_urn="urn:adsk.eagle:package:39191967/2" value="JST2.54X2P" x="22.86" y="11.43" smashed="yes" rot="R180"/>
-<element name="U$5" library="CRD" library_urn="urn:adsk.eagle:library:39051337" package="JST2.54X2P_FOOTPRINT" package3d_urn="urn:adsk.eagle:package:39191967/2" value="JST2.54X2P" x="12.7" y="11.43" smashed="yes" rot="R180"/>
+<element name="U$4" library="CRD" library_urn="urn:adsk.eagle:library:39051337" package="JST2.54X2P_FOOTPRINT" package3d_urn="urn:adsk.eagle:package:39191967/2" value="JST2.54X2P" x="22.86" y="12.065" smashed="yes" rot="R180"/>
+<element name="U$5" library="CRD" library_urn="urn:adsk.eagle:library:39051337" package="JST2.54X2P_FOOTPRINT" package3d_urn="urn:adsk.eagle:package:39191967/2" value="JST2.54X2P" x="12.827" y="12.065" smashed="yes" rot="R180"/>
 <element name="V" library="con-molex" library_urn="urn:adsk.eagle:library:165" package="22-23-2041" package3d_urn="urn:adsk.eagle:package:8078635/1" value="22-23-2041" x="17.78" y="18.796" smashed="yes">
 <attribute name="MF" value="MOLEX" x="17.78" y="18.796" size="1.778" layer="27" display="off"/>
@@
 <contactref element="U$4" pad="1"/>
 <contactref element="U$1" pad="1"/>
-<wire x1="27.94" y1="10.16" x2="26.67" y2="11.43" width="1.5" layer="16"/>
-<wire x1="24.13" y1="11.43" x2="26.67" y2="11.43" width="1.5" layer="16"/>
+<wire x1="27.94" y1="10.16" x2="26.035" y2="12.065" width="1.5" layer="16"/>
+<wire x1="24.13" y1="12.065" x2="26.035" y2="12.065" width="1.5" layer="16"/>
 <wire x1="27.94" y1="10.16" x2="27.94" y2="5.08" width="1.5" layer="16"/>
 <contactref element="V" pad="3"/>
@@
 <contactref element="U$4" pad="2"/>
 <contactref element="U$1" pad="2"/>
-<wire x1="21.59" y1="11.43" x2="21.59" y2="10.77104375" width="1.5" layer="16"/>
+<wire x1="21.59" y1="12.065" x2="21.59" y2="10.77104375" width="1.5" layer="16"/>
 <wire x1="25.4" y1="6.96104375" x2="21.59" y2="10.77104375" width="1.5" layer="16"/>
 <wire x1="25.4" y1="6.96104375" x2="25.4" y2="5.08" width="1.5" layer="16"/>
 <contactref element="V" pad="4"/>
-<wire x1="21.59" y1="11.43" x2="21.59" y2="18.796" width="1.5" layer="16"/>
+<wire x1="21.59" y1="12.065" x2="21.59" y2="18.796" width="1.5" layer="16"/>
 </signal>
 <signal name="V2+">
@@
 <contactref element="U$2" pad="1"/>
 <contactref element="U$3" pad="1"/>
-<wire x1="19.05" y1="5.08" x2="19.05" y2="6.35" width="1.5" layer="16"/>
-<wire x1="19.05" y1="6.35" x2="13.97" y2="11.43" width="1.5" layer="16"/>
+<wire x1="19.05" y1="5.08" x2="19.05" y2="6.731" width="1.5" layer="16"/>
+<wire x1="19.05" y1="6.731" x2="14.097" y2="11.684" width="1.5" layer="16"/>
+<wire x1="14.097" y1="11.684" x2="14.097" y2="12.065" width="1.5" layer="16"/>
 <wire x1="19.05" y1="4.382" x2="17.272" y2="2.604" width="1.5" layer="16"/>
 <wire x1="17.272" y1="2.604" x2="11.366" y2="2.604" width="1.5" layer="16"/>
@@
 <wire x1="19.05" y1="5.08" x2="19.05" y2="4.382" width="1.5" layer="16"/>
 <contactref element="V" pad="2"/>
-<wire x1="13.97" y1="11.43" x2="13.97" y2="13.589" width="1.5" layer="16"/>
-<wire x1="13.97" y1="13.589" x2="16.51" y2="16.129" width="1.5" layer="16"/>
+<wire x1="14.097" y1="12.065" x2="14.097" y2="13.716" width="1.5" layer="16"/>
+<wire x1="14.097" y1="13.716" x2="16.51" y2="16.129" width="1.5" layer="16"/>
 <wire x1="16.51" y1="16.129" x2="16.51" y2="18.796" width="1.5" layer="16"/>
 </signal>
@@
 <contactref element="U$2" pad="2"/>
 <contactref element="U$3" pad="2"/>
-<wire x1="11.43" y1="11.43" x2="11.43" y2="10.16" width="1.5" layer="16"/>
-<wire x1="16.51" y1="5.08" x2="11.43" y2="10.16" width="1.5" layer="16"/>
+<wire x1="11.557" y1="12.065" x2="11.557" y2="10.033" width="1.5" layer="16"/>
+<wire x1="16.51" y1="5.08" x2="11.557" y2="10.033" width="1.5" layer="16"/>
+<wire x1="11.557" y1="10.033" x2="11.43" y2="10.16" width="1.5" layer="16"/>
 <wire x1="11.43" y1="10.16" x2="7.62" y2="6.35" width="1.5" layer="16"/>
 <wire x1="7.62" y1="6.35" x2="7.62" y2="5.08" width="1.5" layer="16"/>
 <contactref element="V" pad="1"/>
-<wire x1="11.43" y1="11.43" x2="11.43" y2="16.256" width="1.5" layer="16"/>
-<wire x1="11.43" y1="16.256" x2="13.97" y2="18.796" width="1.5" layer="16"/>
+<wire x1="11.557" y1="12.065" x2="11.557" y2="16.383" width="1.5" layer="16"/>
+<wire x1="11.557" y1="16.383" x2="13.97" y2="18.796" width="1.5" layer="16"/>
 </signal>
 </signals>
