File: Placa de processamento/Versões/Versão 1/Esquema.brd (EAGLE design)
At the start: 145.1 x 79.8 mm, 17 parts, among them IC1 5V, IC2 5V

Commit message: uptate boards
Parts:
- removed IC1: 5V, v-reg:78XXL
Connections:
- removed net VOUT_LORA: IC1.OUT, U$2.VCC
- net GND: no longer IC1.GND
- net VIN: no longer IC1.IN
- net VOUT: now also U$2.VCC
Routing:
- net VOUT: track 201.8 -> 202.8 mm
Changed lines of the file:
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@@
 <attribute name="VALUE" x="93.7138" y="5.19" size="1.27" layer="27" ratio="10"/>
-</element>
-<element name="IC1" library="v-reg" library_urn="urn:adsk.eagle:library:409" package="78XXL" package3d_urn="urn:adsk.eagle:package:30361/1" value="5V" x="46" y="-18" smashed="yes">
-<attribute name="NAME" x="42.19" y="-12.92" size="1.778" layer="25" ratio="10"/>
-<attribute name="POPULARITY" value="10" x="46" y="-18" size="1.778" layer="27" display="off"/>
-<attribute name="VALUE" x="42.063" y="-15.46" size="1.778" layer="27" ratio="10"/>
 </element>
 </elements>
@@
 <wire x1="15.76" y1="10.29" x2="15.47" y2="10" width="1.5" layer="16"/>
 <wire x1="15.47" y1="10" x2="11" y2="10" width="1.5" layer="16"/>
-<contactref element="IC1" pad="IN"/>
-<wire x1="7.238" y1="9.856" x2="43.46" y2="-21.81" width="0" layer="19" extent="1-1"/>
 </signal>
 <signal name="V_BATTERY">
@@
 <wire x1="137" y1="45.3" x2="143" y2="45.3" width="1.5" layer="1"/>
 <via x="143" y="45.3" extent="1-16" drill="1"/>
-<contactref element="IC1" pad="GND"/>
-<wire x1="128.1" y1="45.3" x2="119.65" y2="75.6" width="0" layer="19" extent="1-1"/>
-<wire x1="125.74" y1="42.13" x2="128.1" y2="45.3" width="0" layer="19" extent="1-1"/>
-<wire x1="94.3488" y1="9" x2="125.74" y2="17.36" width="0" layer="19" extent="1-1"/>
-<wire x1="91" y1="14" x2="94.3488" y2="9" width="0" layer="19" extent="1-1"/>
-<wire x1="75.23" y1="10.16" x2="85" y2="14" width="0" layer="19" extent="1-1"/>
-<wire x1="42.132" y1="18.43" x2="75.23" y2="10.16" width="0" layer="19" extent="1-1"/>
-<wire x1="27.4" y1="17.17" x2="42.132" y2="18.43" width="0" layer="19" extent="1-1"/>
-<wire x1="18.3" y1="10.29" x2="27.4" y2="17.17" width="0" layer="19" extent="1-1"/>
-<wire x1="38.1355" y1="38.0755" x2="27.4" y2="17.17" width="0" layer="19" extent="1-1"/>
-<wire x1="28.829" y1="53.8" x2="38.1355" y2="38.0755" width="0" layer="19" extent="1-1"/>
-<wire x1="56.9" y1="43.8" x2="38.1355" y2="38.0755" width="0" layer="19" extent="1-1"/>
-<wire x1="7.2" y1="35.27" x2="27.4" y2="17.17" width="0" layer="19" extent="1-1"/>
-<wire x1="46" y1="-21.81" x2="18.3" y2="10.29" width="0" layer="19" extent="1-1"/>
 </signal>
 <signal name="N$4">
@@
 <contactref element="U$11" pad="30"/>
 <contactref element="IC2" pad="OUT"/>
-<wire x1="139.1" y1="66.9667875" x2="139.1" y2="67" width="1.5" layer="16"/>
-<wire x1="140.666" y1="65.4007875" x2="139.1" y2="66.9667875" width="1.5" layer="16"/>
+<wire x1="139.5" y1="67" x2="140.766" y2="65.734" width="1.5" layer="16"/>
+<wire x1="140.766" y1="23.846" x2="140.666" y2="23.746" width="1.5" layer="16"/>
 <wire x1="140.666" y1="23.746" x2="134.28" y2="17.36" width="1.5" layer="16"/>
 <wire x1="128.28" y1="17.36" x2="134.28" y2="17.36" width="1.5" layer="16"/>
-<wire x1="140.666" y1="65.4007875" x2="140.666" y2="23.746" width="1.5" layer="16"/>
-<wire x1="139.1" y1="67" x2="138.341" y2="67" width="1.5" layer="16"/>
+<wire x1="140.766" y1="41" x2="140.766" y2="23.846" width="1.5" layer="16"/>
+<wire x1="138.341" y1="67" x2="139.5" y2="67" width="1.5" layer="16"/>
 <wire x1="140.666" y1="23.746" x2="140.666" y2="9.666" width="1.5" layer="16"/>
 <wire x1="140.666" y1="9.666" x2="134" y2="3" width="1.5" layer="16"/>
@@
 <wire x1="20.84" y1="10.29" x2="20.84" y2="6.16" width="1.5" layer="16"/>
 <wire x1="20.84" y1="6.16" x2="24" y2="3" width="1.5" layer="16"/>
+<contactref element="U$2" pad="VCC"/>
+<wire x1="138.303" y1="66.962" x2="138.341" y2="67" width="1.5" layer="16"/>
+<wire x1="140.766" y1="51.766" x2="140" y2="51" width="1.5" layer="16"/>
+<wire x1="140" y1="41.766" x2="140.766" y2="41" width="1.5" layer="16"/>
+<wire x1="140.766" y1="65.734" x2="140.766" y2="51.766" width="1.5" layer="16"/>
+<wire x1="140" y1="51" x2="140" y2="41.766" width="1.5" layer="16"/>
 </signal>
 <signal name="N$7">
 <contactref element="U$2" pad="GND"/>
 <contactref element="R2" pad="2"/>
-<wire x1="132.35" y1="75.6" x2="132.35" y2="75.455" width="1.5" layer="16"/>
+<wire x1="132.35" y1="75.455" x2="132.35" y2="75.6" width="1.5" layer="16"/>
 <wire x1="138.303" y1="69.502" x2="132.35" y2="75.455" width="1.5" layer="16"/>
 </signal>
@@
 <wire x1="105.42" y1="17.36" x2="105.42" y2="20.12" width="1.5" layer="16"/>
 <wire x1="107.562" y1="22.262" x2="122.46095625" y2="22.262" width="1.5" layer="16"/>
-<wire x1="131" y1="55" x2="133" y2="57" width="1.5" layer="16"/>
-<wire x1="133" y1="57" x2="137.3032125" y2="57" width="1.5" layer="16"/>
-<wire x1="137.3032125" y1="57" x2="137.3242125" y2="56.979" width="1.5" layer="16"/>
-<wire x1="137.3242125" y1="56.979" x2="138.126" y2="56.979" width="1.5" layer="16"/>
-<wire x1="138.126" y1="56.979" x2="138.303" y2="56.802" width="1.5" layer="16"/>
 <wire x1="105.42" y1="20.12" x2="107.562" y2="22.262" width="1.5" layer="16"/>
 <wire x1="122.46095625" y1="22.262" x2="131" y2="30.80104375" width="1.5" layer="16"/>
-<wire x1="131" y1="30.80104375" x2="131" y2="55" width="1.5" layer="16"/>
+<wire x1="131" y1="55" x2="131" y2="30.80104375" width="1.5" layer="16"/>
+<wire x1="138.303" y1="56.802" x2="132.802" y2="56.802" width="1.5" layer="16"/>
+<wire x1="132.802" y1="56.802" x2="131" y2="55" width="1.5" layer="16"/>
 </signal>
 <signal name="M0">
@@
 <contactref element="U$1" pad="SCL"/>
 <contactref element="U$9" pad="SCL"/>
-<wire x1="40.7355" y1="38.0755" x2="40.7355" y2="22.3665" width="1.5" layer="16"/>
-<wire x1="44.672" y1="18.43" x2="40.7355" y2="22.3665" width="1.5" layer="16"/>
+<wire x1="40.7355" y1="38.0755" x2="40.7355" y2="25.3665" width="1.5" layer="16"/>
+<wire x1="44.672" y1="18.43" x2="44.672" y2="21.43" width="1.5" layer="16"/>
+<wire x1="44.672" y1="21.43" x2="40.7355" y2="25.3665" width="1.5" layer="16"/>
 <wire x1="40.7355" y1="38.0755" x2="40.7355" y2="39.7355" width="1.5" layer="16"/>
 <wire x1="40.7355" y1="39.7355" x2="42.378" y2="41.378" width="1.5" layer="16"/>
@@
 <contactref element="U$11" pad="10"/>
 <contactref element="U$8" pad="MISO"/>
-<wire x1="28.829" y1="51.26" x2="103.74" y2="51.26" width="1.5" layer="16"/>
-<wire x1="105.42" y1="49.58" x2="105.42" y2="42.13" width="1.5" layer="16"/>
-<wire x1="103.74" y1="51.26" x2="105.42" y2="49.58" width="1.5" layer="16"/>
+<wire x1="28.829" y1="51.26" x2="104.14" y2="51.26" width="1.5" layer="16"/>
+<wire x1="105.42" y1="49.98" x2="105.42" y2="42.13" width="1.5" layer="16"/>
+<wire x1="104.14" y1="51.26" x2="105.42" y2="49.98" width="1.5" layer="16"/>
 </signal>
 <signal name="CS">
@@
 <wire x1="103" y1="17.24" x2="102.88" y2="17.36" width="1.5" layer="16"/>
 <wire x1="123.47" y1="7.82" x2="123.47" y2="8.53" width="1.5" layer="16"/>
-<wire x1="106.1" y1="11.9" x2="103" y2="15" width="1.5" layer="16"/>
-<wire x1="123.47" y1="8.53" x2="120.1" y2="11.9" width="1.5" layer="16"/>
-<wire x1="120.1" y1="11.9" x2="106.1" y2="11.9" width="1.5" layer="16"/>
+<wire x1="106.4" y1="11.6" x2="103" y2="15" width="1.5" layer="16"/>
+<wire x1="123.47" y1="8.53" x2="120.4" y2="11.6" width="1.5" layer="16"/>
+<wire x1="120.4" y1="11.6" x2="106.4" y2="11.6" width="1.5" layer="16"/>
 </signal>
 <signal name="OPTOACOPLADOR2">
@@
 <contactref element="U$5" pad="2"/>
 <wire x1="100.34" y1="14" x2="100.34" y2="17.36" width="1.5" layer="16"/>
-<wire x1="100.34" y1="14" x2="104.702" y2="9.638" width="1.5" layer="16"/>
-<wire x1="119.112" y1="9.638" x2="120.93" y2="7.82" width="1.5" layer="16"/>
-<wire x1="104.702" y1="9.638" x2="119.112" y2="9.638" width="1.5" layer="16"/>
-</signal>
-<signal name="VOUT_LORA">
-<contactref element="IC1" pad="OUT"/>
-<contactref element="U$2" pad="VCC"/>
-<wire x1="48.54" y1="-21.81" x2="138.303" y2="66.962" width="0" layer="19" extent="1-1"/>
+<wire x1="100.34" y1="14" x2="105.202" y2="9.138" width="1.5" layer="16"/>
+<wire x1="119.612" y1="9.138" x2="120.93" y2="7.82" width="1.5" layer="16"/>
+<wire x1="105.202" y1="9.138" x2="119.612" y2="9.138" width="1.5" layer="16"/>
 </signal>
 </signals>
