File: Placa de processamento/Versões/Versão 2/Esquema.brd (EAGLE design)
At the start: 145.1 x 79.8 mm, 17 parts, among them IC1 5V, IC2 5V

Commit message: update position
Parts:
- moved IC1 1.32 mm to (15.2, 33.3)
- moved R1 1.30 mm to (18.0, 41.3)
- moved U$8 1.13 mm to (21.2, 52.5)
Routing:
- net VIN: track 79.5 -> 80.8 mm
- net 3V3: track 176.6 -> 177.8 mm
- net LED1: track 133.8 -> 132.6 mm
- net VOUT_LORA: track 166.6 -> 167.7 mm
- net MOSI: track 68.3 -> 69.1 mm
- net MISO: track 86.5 -> 87.4 mm
- net CLK: track 87.3 -> 88.2 mm
